File: PCB Design/Power Distribution/Power Distribution.kicad_pcb (KiCad board)
At the start: 2 copper layers, 83.3 x 44.3 mm, 27 parts, among them J1 Barrel_Jack, J2 Barrel_Jack, J3 Barrel_Jack, J4 Barrel_Jack, J5 Barrel_Jack, J6 Switch Header Pin, J7 LED, Q1 2N7002, Q2 NCE30P30K, Q3 2N7002

Commit message: $1
Parts:
- added J8: Conn_01x02_Pin, Connector_PinHeader_2.54mm:PinHeader_1x02_P2.54mm_Vertical, F.Cu at (212.2, 116.8)
- added J9: Conn_01x02_Pin, Connector_PinHeader_2.54mm:PinHeader_1x02_P2.54mm_Vertical, F.Cu at (212.2, 122.0)
- J6: footprint Footprints:3 Pin Male Header -> Connector_PinHeader_2.54mm:PinHeader_1x03_P2.54mm_Vertical; moved to F.Cu
- J7: moved to F.Cu
- Q2: footprint Footprints:NCE30P30K P channel MOSFET -> Package_TO_SOT_SMD:TO-252-2
- TP1, TP2, TP3: footprint TestPoint:TestPoint_Plated_Hole_D2.0mm -> TestPoint:TestPoint_THTPad_D1.0mm_Drill0.5mm
- moved D2 25.2 mm to (238.7, 126.6), turned to -90 degrees
- moved C4 22.1 mm to (251.8, 129.0)
- moved R1 19.2 mm to (244.8, 109.8), turned to 0 degrees
- moved Q2 18.7 mm to (246.6, 120.6)
- moved TP1 18.5 mm to (242.5, 104.0), turned to 90 degrees
- moved TP2 18.5 mm to (246.8, 104.0), turned to 90 degrees
- moved TP3 18.5 mm to (251.0, 104.0), turned to 90 degrees
- moved C3 17.8 mm to (244.8, 111.3), turned to 0 degrees
- moved J3 17.8 mm to (257.9, 105.9)
- moved J5 17.8 mm to (257.9, 133.9)
- moved F2 17.7 mm to (220.9, 130.3)
- moved J2 17.7 mm to (199.5, 133.9)
- moved J4 17.5 mm to (257.9, 120.2)
- moved D1 17.5 mm to (238.7, 111.9)
- moved J1 17.4 mm to (199.5, 111.8)
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Routing:
- net /Supply: track 48.2 -> 25.5 mm
- net /Mains: track 29.4 -> 45.7 mm
- net Net-(J7-Pin_2): track 6.27 -> 21.3 mm
- net /Vout: track 59.5 -> 68.9 mm, vias 1 -> 0
- net /Battery output: track 21.3 -> 15.5 mm
- net /AC/DC output: track 21.0 -> 15.7 mm
- net /Switch: track 50.8 -> 56.0 mm
- net /Battery: track 29.4 -> 24.5 mm
- net Net-(Q2-G): track 33.3 -> 35.9 mm
- net Net-(Q1-G): track 14.4 -> 12.2 mm
- net GND: vias 0 -> 1
Other:
- board size 83.3 x 44.3 mm -> 83 x 46 mm
- board text added: "Designed by Sarah Tallack June 2023"
- board text added: "LED"
- board text added: "Out"
- board text added: "S1"
- board text added: "S2"
- board text added: "Version 2"
- board text removed: "8A Fuse"
- board text removed: "Based off of design by Stanton (2022)"
- board text removed: "Designed by Sarah Tallack December 2022"
- board text removed: "GND"
- board text removed: "LED Indicator"
- board text removed: "Output"
- board text removed: "Power Distribution for Sea Ice Imaging Rig V0"
- board text removed: "SIIR"
- board text removed: "V+"

Commit message: $1
Other:
- board text added: "Version 1"
- board text removed: "Version 2"
Changed lines of the file:
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@@
     (descr "Through hole straight pin header, 1x02, 2.54mm pitch, single row")
     (tags "Through hole pin header THT 1x02 2.54mm single row")
+    (property "Populate" "0")
     (property "Sheetfile" "Power Distribution.kicad_sch")
     (property "Sheetname" "")
@@
     (fp_line (start 1 0.625) (end -1 0.625)
       (stroke (width 0.1) (type solid)) (layer "F.Fab"))
-    (pad "1" smd roundrect (at -0.9125 0 90) (size 1.025 1.4) (layers "F.Cu" "F.Paste" "F.Mask") (roundrect_rratio 0.243902)
+    (pad "1" smd roundrect (at -0.9125 0 90) (size 1.025 1.4) (layers "F.Cu" "F.Paste" "F.Mask") (roundrect_rratio 0.243902439)
       (net 12 "Net-(Q2-G)") (pintype "passive"))
-    (pad "2" smd roundrect (at 0.9125 0 90) (size 1.025 1.4) (layers "F.Cu" "F.Paste" "F.Mask") (roundrect_rratio 0.243902)
+    (pad "2" smd roundrect (at 0.9125 0 90) (size 1.025 1.4) (layers "F.Cu" "F.Paste" "F.Mask") (roundrect_rratio 0.243902439)
       (net 15 "Net-(Q1-D)") (pintype "passive"))
     (model "${KICAD6_3DMODEL_DIR}/Resistor_SMD.3dshapes/R_0805_2012Metric.wrl"
@@
     (fp_line (start 1 0.625) (end -1 0.625)
       (stroke (width 0.1) (type solid)) (layer "F.Fab"))
-    (pad "1" smd roundrect (at -0.9125 0 270) (size 1.025 1.4) (layers "F.Cu" "F.Paste" "F.Mask") (roundrect_rratio 0.243902)
+    (pad "1" smd roundrect (at -0.9125 0 270) (size 1.025 1.4) (layers "F.Cu" "F.Paste" "F.Mask") (roundrect_rratio 0.243902439)
       (net 16 "Net-(Q3-D)") (pintype "passive"))
-    (pad "2" smd roundrect (at 0.9125 0 270) (size 1.025 1.4) (layers "F.Cu" "F.Paste" "F.Mask") (roundrect_rratio 0.243902)
+    (pad "2" smd roundrect (at 0.9125 0 270) (size 1.025 1.4) (layers "F.Cu" "F.Paste" "F.Mask") (roundrect_rratio 0.243902439)
       (net 13 "Net-(J7-Pin_2)") (pintype "passive"))
     (model "${KICAD6_3DMODEL_DIR}/Resistor_SMD.3dshapes/R_0805_2012Metric.wrl"
@@
     (fp_line (start 1.6 0.8) (end -1.6 0.8)
       (stroke (width 0.1) (type solid)) (layer "F.Fab"))
-    (pad "1" smd roundrect (at -1.475 0 180) (size 1.15 1.8) (layers "F.Cu" "F.Paste" "F.Mask") (roundrect_rratio 0.217391)
+    (pad "1" smd roundrect (at -1.475 0 180) (size 1.15 1.8) (layers "F.Cu" "F.Paste" "F.Mask") (roundrect_rratio 0.2173913043)
       (net 4 "/Vout") (pintype "passive"))
-    (pad "2" smd roundrect (at 1.475 0 180) (size 1.15 1.8) (layers "F.Cu" "F.Paste" "F.Mask") (roundrect_rratio 0.217391)
+    (pad "2" smd roundrect (at 1.475 0 180) (size 1.15 1.8) (layers "F.Cu" "F.Paste" "F.Mask") (roundrect_rratio 0.2173913043)
       (net 2 "GND") (pintype "passive"))
     (model "${KICAD6_3DMODEL_DIR}/Capacitor_SMD.3dshapes/C_1206_3216Metric.wrl"
@@
   (footprint "Footprints:2 Pin Male Header" (layer "F.Cu")
     (at 228.791746 139.683984 180)
-    (property "Extended" "1")
-    (property "LCSC" "C20079")
-    (property "Populate" "1")
-    (property "Price" "0.0058")
+    (property "Extended" "")
+    (property "LCSC" "")
+    (property "Populate" "0")
+    (property "Price" "")
     (property "Sheetfile" "Power Distribution.kicad_sch")
     (property "Sheetname" "")
@@
     (descr "Through hole straight pin header, 1x02, 2.54mm pitch, single row")
     (tags "Through hole pin header THT 1x02 2.54mm single row")
+    (property "Populate" "0")
     (property "Sheetfile" "Power Distribution.kicad_sch")
     (property "Sheetname" "")
@@
     (tags "Through hole pin header THT 1x03 2.54mm single row")
     (property "Extended" "")
-    (property "LCSC" "C20547")
+    (property "LCSC" "")
     (property "Populate" "0")
     (property "Price" "")
@@
     (fp_line (start 4.11 2.7) (end 3.11 2.7)
       (stroke (width 0.1) (type solid)) (layer "F.Fab"))
-    (pad "1" smd roundrect (at -5.04 -2.28 270) (size 2.2 1.2) (layers "F.Cu" "F.Paste" "F.Mask") (roundrect_rratio 0.208333)
+    (pad "1" smd roundrect (at -5.04 -2.28 270) (size 2.2 1.2) (layers "F.Cu" "F.Paste" "F.Mask") (roundrect_rratio 0.2083333333)
       (net 12 "Net-(Q2-G)") (pinfunction "G") (pintype "passive"))
-    (pad "2" smd roundrect (at -0.415 -1.525 270) (size 3.05 2.75) (layers "F.Cu" "F.Paste") (roundrect_rratio 0.090909)
+    (pad "2" smd roundrect (at -0.415 -1.525 270) (size 3.05 2.75) (layers "F.Cu" "F.Paste") (roundrect_rratio 0.09090909091)
       (net 4 "/Vout") (pinfunction "D") (pintype "passive"))
-    (pad "2" smd roundrect (at -0.415 1.525 270) (size 3.05 2.75) (layers "F.Cu" "F.Paste") (roundrect_rratio 0.090909)
+    (pad "2" smd roundrect (at -0.415 1.525 270) (size 3.05 2.75) (layers "F.Cu" "F.Paste") (roundrect_rratio 0.09090909091)
       (net 4 "/Vout") (pinfunction "D") (pintype "passive"))
-    (pad "2" smd roundrect (at 1.26 0 270) (size 6.4 5.8) (layers "F.Cu" "F.Mask") (roundrect_rratio 0.043103)
+    (pad "2" smd roundrect (at 1.26 0 270) (size 6.4 5.8) (layers "F.Cu" "F.Mask") (roundrect_rratio 0.04310293103)
       (net 4 "/Vout") (pinfunction "D") (pintype "passive"))
-    (pad "2" smd roundrect (at 2.935 -1.525 270) (size 3.05 2.75) (layers "F.Cu" "F.Paste") (roundrect_rratio 0.090909)
+    (pad "2" smd roundrect (at 2.935 -1.525 270) (size 3.05 2.75) (layers "F.Cu" "F.Paste") (roundrect_rratio 0.09090909091)
       (net 4 "/Vout") (pinfunction "D") (pintype "passive"))
-    (pad "2" smd roundrect (at 2.935 1.525 270) (size 3.05 2.75) (layers "F.Cu" "F.Paste") (roundrect_rratio 0.090909)
+    (pad "2" smd roundrect (at 2.935 1.525 270) (size 3.05 2.75) (layers "F.Cu" "F.Paste") (roundrect_rratio 0.09090909091)
       (net 4 "/Vout") (pinfunction "D") (pintype "passive"))
-    (pad "3" smd roundrect (at -5.04 2.28 270) (size 2.2 1.2) (layers "F.Cu" "F.Paste" "F.Mask") (roundrect_rratio 0.208333)
+    (pad "3" smd roundrect (at -5.04 2.28 270) (size 2.2 1.2) (layers "F.Cu" "F.Paste" "F.Mask") (roundrect_rratio 0.2083333333)
       (net 3 "/Supply") (pinfunction "S") (pintype "passive"))
     (model "${KICAD6_3DMODEL_DIR}/Package_TO_SOT_SMD.3dshapes/TO-252-2.wrl"
@@
     (effects (font (size 1 1) (thickness 0.15)) (justify mirror))
   )
-  (gr_text "Version 2" (at 196.5 144) (layer "B.SilkS")
+  (gr_text "Version 1" (at 196.5 144) (layer "B.SilkS")
     (effects (font (size 1 1) (thickness 0.15)) (justify left mirror))
   )
@@
     (effects (font (size 1 1) (thickness 0.15)) (justify right mirror))
   )
-  (gr_text "Power Distribution for \nSea Ice Imaging Rig" (at 250.25 135.5) (layer "B.SilkS")
+  (gr_text "Power Distribution for \nSea Ice Imaging Rig" (at 250 118.25) (layer "B.SilkS")
     (effects (font (size 1 1) (thickness 0.15)) (justify left mirror))
   )
@@
     (effects (font (size 1 1) (thickness 0.15)) (justify mirror))
   )
-  (gr_text "LED" (at 232.75 136) (layer "B.SilkS")
+  (gr_text "LED" (at 231.5 136) (layer "B.SilkS")
     (effects (font (size 1 1) (thickness 0.15)) (justify left mirror))
   )
-  (gr_text "Designed by Sarah Tallack \nJune 2023" (at 250.25 138.75) (layer "B.SilkS")
-    (effects (font (size 0.75 0.75) (thickness 0.15)) (justify left mirror))
+  (gr_text "Designed by Sarah Tallack \nJune 2023" (at 250 121.75) (layer "B.SilkS")
+    (effects (font (size 0.8 0.8) (thickness 0.15)) (justify left mirror))
   )
   (gr_text "Output 3" (at 266.75 136.25 90) (layer "B.SilkS")
@@
     (effects (font (size 0.8 0.8) (thickness 0.15)))
   )
-  (gr_text "Version 2" (at 189 144.25) (layer "F.SilkS")
+  (gr_text "Version 1" (at 189 144.25) (layer "F.SilkS")
     (effects (font (size 1 1) (thickness 0.15)) (justify left))
   )
@@
   )
   (gr_text "Designed by Sarah Tallack \nJune 2023" (at 234 139) (layer "F.SilkS")
-    (effects (font (size 0.75 0.75) (thickness 0.15)) (justify left))
+    (effects (font (size 0.8 0.8) (thickness 0.15)) (justify left))
   )
   (gr_text "S2" (at 218.75 136.25) (layer "F.SilkS")
@@
     (effects (font (size 1 1) (thickness 0.15)) (justify left))
   )
-  (dimension (type aligned) (layer "F.SilkS")
-    (pts (xy 266 99.75) (xy 266 145.75))
-    (height -16)
-    (gr_text "46,0000 mm" (at 280.85 122.75 90) (layer "F.SilkS")
-      (effects (font (size 1 1) (thickness 0.15)))
-    )
-    (format (prefix "") (suffix "") (units 3) (units_format 1) (precision 4))
-    (style (thickness 0.15) (arrow_length 1.27) (text_position_mode 0) (extension_height 0.58642) (extension_offset 0.5) keep_text_aligned)
-  )
   (segment (start 209.613132 108.239131) (end 209.624001 108.25) (width 3.6) (layer "F.Cu") (net 1))
