File: PCB Design/Power Distribution/Power Distribution.kicad_sch (KiCad schematic)
At the start: 27 parts, among them J1 Barrel_Jack, J2 Barrel_Jack, J3 Barrel_Jack, J4 Barrel_Jack, J5 Barrel_Jack, J6 Switch Header Pin, J7 LED, Q1 2N7002, Q2 NCE30P30K, Q3 2N7002

Commit message: $1
Parts:
- added J8, J9: Conn_01x02_Pin, Connector_PinHeader_2.54mm:PinHeader_1x02_P2.54mm_Vertical, symbol Connector:Conn_01x02_Pin
- C1, C2: LCSC (none) -> C15195; LCSC No. C15195 -> (none); Populate Yes -> 1
- C3: LCSC (none) -> C307331; LCSC No. C307331 -> (none); Populate Yes -> 1
- C4: LCSC (none) -> C29823; LCSC No. C29823 -> (none); Populate (none) -> 1
- D1, D2: LCSC (none) -> C65020; LCSC No. C65020 -> (none); Populate (none) -> 1
- F1, F2: LCSC (none) -> C3131; LCSC No. C3131 -> (none); Populate (none) -> 1
- J1, J2: LCSC (none) -> C98732; LCSC No. C98732 -> (none); Populate (none) -> 1
- J3, J4, J5: LCSC (none) -> C388625; LCSC No. C388625 -> (none); Populate (none) -> 1
- J6: footprint Footprints:3 Pin Male Header -> Connector_PinHeader_2.54mm:PinHeader_1x03_P2.54mm_Vertical; Extended 1 -> (none); LCSC (none) -> C20547; LCSC No. C20547 -> (none); Populate (none) -> 0; Price 0.0303 -> (none)
- J7: LCSC (none) -> C20079; LCSC No. C20079 -> (none); Populate (none) -> 1
- Q1, Q3: LCSC (none) -> C8545; LCSC No. C8545 -> (none); Populate (none) -> 1
- Q2: footprint Footprints:NCE30P30K P channel MOSFET -> Package_TO_SOT_SMD:TO-252-2; LCSC (none) -> C130106; LCSC No. C130106 -> (none); Populate (none) -> 1
- R1: LCSC (none) -> C25778; LCSC No. C25778 -> (none); Populate (none) -> 1
- R2: LCSC (none) -> C25744; LCSC No. C25744 -> (none); Populate (none) -> 1
- R3, R5: LCSC (none) -> C25741; LCSC No. C25741 -> (none); Populate (none) -> 1
- R4: LCSC (none) -> C17840; LCSC No. C17840 -> (none); Populate (none) -> 1
- R6: LCSC (none) -> C17398; LCSC No. C17398 -> (none); Populate (none) -> 1
- TP1, TP2, TP3: footprint TestPoint:TestPoint_Plated_Hole_D2.0mm -> TestPoint:TestPoint_THTPad_D1.0mm_Drill0.5mm
Connections:
- net AC/DC output: now also J8.2 (Pin_2)
- net Battery output: now also J9.2 (Pin_2)
- net GND: now also J8.1 (Pin_1), J9.1 (Pin_1)
Other:
- moved on the sheet: C2, F1, F2, J2

Commit message: $1
Parts:
- J6: LCSC C20547 -> (none)
- J7: Extended 1 -> (none); LCSC C20079 -> (none); Populate 1 -> 0; Price 0.0058 -> (none)
- J8, J9: Populate (none) -> 0
Changed lines of the file:
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@@
       (effects (font (size 1.27 1.27)) hide)
     )
-    (property "LCSC" "C20547" (at 120.65 39.37 0)
+    (property "LCSC" "" (at 120.65 39.37 0)
       (effects (font (size 1.27 1.27)) hide)
     )
@@
       (effects (font (size 1.27 1.27)) hide)
     )
-    (property "Datasheet" "https://datasheet.lcsc.com/lcsc/1811132110_BOOMELE-Boom-Precision-Elec-XH-2A_C20079.pdf" (at 63.5 100.33 0)
-      (effects (font (size 1.27 1.27)) hide)
-    )
-    (property "Price" "0.0058" (at 63.5 100.33 0)
-      (effects (font (size 1.27 1.27)) hide)
-    )
-    (property "Extended" "1" (at 63.5 100.33 0)
-      (effects (font (size 1.27 1.27)) hide)
-    )
-    (property "LCSC" "C20079" (at 63.5 100.33 0)
-      (effects (font (size 1.27 1.27)) hide)
-    )
-    (property "Populate" "1" (at 63.5 100.33 0)
+    (property "Datasheet" "" (at 63.5 100.33 0)
+      (effects (font (size 1.27 1.27)) hide)
+    )
+    (property "Price" "" (at 63.5 100.33 0)
+      (effects (font (size 1.27 1.27)) hide)
+    )
+    (property "Extended" "" (at 63.5 100.33 0)
+      (effects (font (size 1.27 1.27)) hide)
+    )
+    (property "LCSC" "" (at 63.5 100.33 0)
+      (effects (font (size 1.27 1.27)) hide)
+    )
+    (property "Populate" "0" (at 63.5 100.33 0)
       (effects (font (size 1.27 1.27)) hide)
     )
@@
     )
     (property "Datasheet" "~" (at 45.72 22.86 0)
+      (effects (font (size 1.27 1.27)) hide)
+    )
+    (property "Populate" "0" (at 45.72 22.86 0)
       (effects (font (size 1.27 1.27)) hide)
     )
@@
       (effects (font (size 1.27 1.27)) hide)
     )
+    (property "Populate" "0" (at 45.72 52.07 0)
+      (effects (font (size 1.27 1.27)) hide)
+    )
