File: PCB Design/Temperature Controller/Temperature Controller.kicad_pcb (KiCad board)
At the start: 2 copper layers, 70 x 55 mm, 32 parts, among them J1 PT100 Header Pins, J2 Switch Header Pins, J3 LED Header Pins, J5 Barrel_Jack, J6 Conn_01x19_Female, J7 Conn_01x19_Female, J8 Conn_01x03_Male, K1 SANYOU_SRD_Form_C, Q3 S8050_SMD, U1 INA826AIDR

Commit message: $1
Parts:
- removed C1, C2: 100n, Capacitor_SMD:C_0603_1608Metric
- added R13: 13k, Resistor_SMD:R_0603_1608Metric, F.Cu at (143.4, 100.3)
- added R14: 4.3k, Resistor_SMD:R_0603_1608Metric, F.Cu at (145.1, 100.3)
- added R7: 1.1k, Resistor_SMD:R_0603_1608Metric, F.Cu at (145.2, 91.1)
- added R8: 10k, Resistor_SMD:R_0603_1608Metric, F.Cu at (139.0, 93.9)
- added U2: CJ431, Package_TO_SOT_SMD:SOT-23, F.Cu at (140.2, 100.2)
- C4, D1, D2, Q3: moved to F.Cu
- R1, R2, R4: footprint Resistor_SMD:R_0402_1005Metric -> Resistor_SMD:R_0603_1608Metric
- R11, R12, R6: footprint Resistor_SMD:R_0402_1005Metric -> Resistor_SMD:R_0603_1608Metric; moved to F.Cu
- R5: value 300 -> 27k
- U1: value INA826AIDR -> INA332; footprint Footprints:INA826AIDR Instrumentation Amplifier -> Package_SO:VSSOP-8_3.0x3.0mm_P0.65mm
- moved J5 35.5 mm to (157.1, 94.1), turned to 90 degrees
- moved TP4 25.7 mm to (154.0, 63.2)
- moved TP7 19.0 mm to (122.8, 88.2)
- moved TP6 18.5 mm to (116.2, 88.5)
- moved TP9 17.0 mm to (144.2, 82.5), turned to 90 degrees
- moved R12 14.4 mm to (141.5, 62.5), turned to -90 degrees
- moved TP8 14.1 mm to (136.8, 85.5), turned to 90 degrees
- moved U1 12.9 mm to (142.1, 92.5)
- moved TP1 11.6 mm to (146.0, 58.1)
- moved TP5 11.0 mm to (152.5, 82.8)
- moved TP2 10.7 mm to (146.0, 65.8)
- moved TP3 10.3 mm to (146.0, 72.0)
- moved J2 10.2 mm to (121.8, 99.7)
- moved Q3 9.94 mm to (138.2, 62.6)
- moved R5 9.66 mm to (147.0, 91.1)
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Connections:
- D2 pad 2: Net-(R11-Pad1) -> Net-(D2-A)
- J5 pad 1: /COM -> /VIN
- J5 pad 2: /NO -> GND
- R11 pad 1: Net-(R11-Pad1) -> /+5V
- R11 pad 2: /+5V -> Net-(D2-A)
- R5 pad 1: Net-(R5-Pad1) -> Net-(U1-RG)
- R5 pad 2: Net-(R5-Pad2) -> /PC0
- U1 pad 1: /Vb -> Net-(U1-RG)
- U1 pad 2: Net-(R5-Pad1) -> /Vb
- U1 pad 3: Net-(R5-Pad2) -> /Va
- U1 pad 4: /Va -> GND
- U1 pad 5: GND -> /Vref
- U1 pad 6: GND -> /PC0
- U1 pad 7: /PC0 -> /+3V3
- U1 pad 8: /+3V3 -> /PC1
Routing:
- net /PD2: track 81.4 -> 24.3 mm
- net /+3V3: track 52.1 -> 79.1 mm, vias 0 -> 2
- net /PC1: track 0.00 -> 23.3 mm
- net /NO: track 34.6 -> 12.1 mm
- net /PB5: track 30.7 -> 12.1 mm
- net /COM: track 68.4 -> 52.9 mm
- net /Vref: track 0.00 -> 14.6 mm
- net /VIN: track 0.00 -> 12.1 mm
- net Net-(J3-Pin_1): track 13.7 -> 5.77 mm
- net /PB3: track 43.0 -> 36.7 mm
- net /+5V: track 61.4 -> 67.4 mm
- net /Va: track 27.5 -> 21.9 mm, vias 0 -> 1
- net Net-(D1-A): track 28.3 -> 32.5 mm
- net Net-(U2-REF): track 0.00 -> 4.02 mm
- net Net-(U1-RG): track 0.00 -> 3.91 mm
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Other:
- outline, holes or cut-outs redrawn
- board text added: "Designed by Sarah Tallack Jube 2023"
- board text added: "Designed by Sarah Tallack June 2023"
- board text added: "LED"
- board text added: "V1"
- board text removed: "Designed by Sarah Tallack Decmember 2022"
- board text removed: "LED Indicator"
- board text removed: "V0"
