File: PCB Design/Temperature Controller/Temperature Controller.kicad_sch (KiCad schematic)
At the start: 32 parts, among them J1 PT100 Header Pins, J2 Switch Header Pins, J3 LED Header Pins, J5 Barrel_Jack, J6 Conn_01x19_Female, J7 Conn_01x19_Female, J8 Conn_01x03_Male, K1 SANYOU_SRD_Form_C, Q3 S8050_SMD, U1 INA826AIDR

Commit message: $1
Parts:
- removed C1, C2: 100n, Capacitor_SMD:C_0603_1608Metric, symbol Device:C_Small
- removed R11: 1.2k, Resistor_SMD:R_0402_1005Metric, symbol Device:R_Small_US
- added R11: 1.2k, Resistor_SMD:R_0603_1608Metric, symbol Device:R
- added R13: 13k, Resistor_SMD:R_0603_1608Metric, symbol Device:R
- added R14: 4.3k, Resistor_SMD:R_0603_1608Metric, symbol Device:R
- added R7: 1.1k, Resistor_SMD:R_0603_1608Metric, symbol Device:R
- added R8: 10k, Resistor_SMD:R_0603_1608Metric, symbol Device:R
- added U2: CJ431, Package_TO_SOT_SMD:SOT-23, symbol Reference_Voltage:CJ432
- C4: LCSC No. C96446 -> (none); Populate Yes -> 1
- D1: LCSC No. C8598 -> (none); Populate Yes -> 1
- D2: Populate Yes -> 1
- J1, J2, J3: Extended (none) -> 1; LCSC No. C20079 -> (none); Populate (none) -> 1
- J5: Extended (none) -> 1; LCSC No. C388625 -> (none); Populate (none) -> 1
- J6, J7: Populate (none) -> 0
- J8: LCSC No. C72334 -> (none); Populate Yes -> 1
- K1: LCSC No. C35449 -> (none); Populate Yes -> 1
- Q3: LCSC No. C2146 -> (none); Populate Yes -> 1
- R1, R2: footprint Resistor_SMD:R_0402_1005Metric -> Resistor_SMD:R_0603_1608Metric; LCSC C25890 -> C22978; LCSC No. C26010 -> (none); Populate Yes -> 1
- R12: footprint Resistor_SMD:R_0402_1005Metric -> Resistor_SMD:R_0603_1608Metric; LCSC C25862 -> C22765; LCSC No. C25862 -> (none); Populate Yes -> 1
- R3: LCSC No. C543443 -> (none); Populate Yes -> 1
- R4: footprint Resistor_SMD:R_0402_1005Metric -> Resistor_SMD:R_0603_1608Metric; LCSC C25862 -> C22765; LCSC No. C17398 -> (none); Populate Yes -> 1; now left out of the parts list
- R5: value 300 -> 27k; Extended 1 -> 0; LCSC C352332 -> C22967; LCSC No. C17617 -> (none); Populate Yes -> 1; Price 0.0027 -> 0.0016
- R6: footprint Resistor_SMD:R_0402_1005Metric -> Resistor_SMD:R_0603_1608Metric; LCSC C25862 -> C22765; LCSC No. C17398 -> (none); Populate Yes -> 1
- U1: value INA826AIDR -> INA332; footprint Footprints:INA826AIDR Instrumentation Amplifier -> Package_SO:VSSOP-8_3.0x3.0mm_P0.65mm; LCSC C38433 -> C181461; LCSC No. C38433 -> (none)
Connections:
- net +3V3: now also U1.7 (V+), R8.1; no longer U1.8 (Vs+)
- net +5V: now also R11.1
- net COM: no longer J5.1
- net GND: now also J5.2, U1.4 (V-), R14.2, U2.3 (A); no longer U1.5 (Vs-), U1.6 (Ref)
- net NO: no longer J5.2
- net PC0: now also R5.2, U1.6; no longer U1.7
- net PC1: now also U1.8 (SD)
- net VIN: now also J5.1
- net Va: now also U1.3 (+); no longer U1.4 (+)
- net Vb: now also U1.2 (-); no longer U1.1 (-)
- net at R5.1: now also U1.1 (RG), R7.1; no longer U1.2 (Rg)
- net at D2.2 (A): now also R11.2
- new net: R13.2, R14.1, U2.1 (REF)
- new net Vref: R13.1, R7.2, R8.2, U1.5 (Ref), U2.2 (K)
Other:
- note added: "ADC input"
- note added: "Button Input"
- note added: "GPIO output"
- note added: "Heater Output"
- note added: "LED output"
- note added: "UART"
- note added: "Voltage Reference for Instrumentation Amplifier"
- note removed: "Max Current Draw from battery: - From heating pads ~ about 2A - Barrel jack/ Power connector with 5A rating at >=12V should be enough"
- moved on the sheet: C4, J2, J3, J5, R1, R2, R4, R6, TP1, TP2, TP3, TP4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

Commit message: $1
Parts:
- R3: LCSC C101397 -> C2960792
Changed lines of the file:
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@@
       (effects (font (size 1.27 1.27)) hide)
     )
-    (property "LCSC" "C101397" (at 41.91 45.72 0)
+    (property "LCSC" "C2960792" (at 41.91 45.72 0)
       (effects (font (size 1.27 1.27)) hide)
     )
